File: PCB Schematics/LEDMatrix/LEDMatrix.kicad_pcb (KiCad board)
At the start: 2 copper layers, 49.9 x 124.7 mm, 25 parts, among them J1 Conn_01x02, P1 Digital, SW1 SW_Push, SW2 SW_Push, SW3 SW_Push, SW4 SW_Push, SW5 SW_Push, U1 74HC595, U2 74HC595, U3 LED8x8Matrix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

Commit message: Changing README
Other:
- board text removed: "alright have fun kids"
Changed lines of the file:
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@@
-(kicad_pcb (version 20171130) (host pcbnew "(5.1.0)-1")
+(kicad_pcb (version 20171130) (host pcbnew "(5.1.5)-3")
   (general
     (thickness 1.6)
-    (drawings 99)
+    (drawings 98)
     (tracks 524)
     (zones 0)
@@
   (page A4)
   (layers
-    (0 F.Cu signal)
-    (31 B.Cu signal)
-    (32 B.Adhes user hide)
-    (33 F.Adhes user hide)
-    (34 B.Paste user hide)
-    (35 F.Paste user hide)
-    (36 B.SilkS user hide)
-    (37 F.SilkS user hide)
+    (0 F.Cu signal hide)
+    (31 B.Cu signal hide)
+    (32 B.Adhes user)
+    (33 F.Adhes user)
+    (34 B.Paste user)
+    (35 F.Paste user)
+    (36 B.SilkS user)
+    (37 F.SilkS user)
     (38 B.Mask user hide)
     (39 F.Mask user hide)
@@
     )
   )
-  (gr_text "alright have fun kids\n" (at 73.9394 78.1304) (layer F.SilkS)
-    (effects (font (size 1 1) (thickness 0.15)))
-  )
   (gr_text "Edwin L." (at 38.227 77.1652) (layer F.SilkS)
